Commit message: [change] Project name and an old ros launch file

File: taylor_robot_description/urdf/Taylor_URDF_assembly.urdf (robot description, URDF)
Before this commit: robot Taylor_URDF_assembly, 5 links, 4 joints
Links:
- link base_link: geometry collision mesh filename=package://taylor_description/meshes/base_link.STL; visual mesh filename=package://taylor_description/meshes/base_link.STL
- link caster_wheel: geometry collision mesh filename=package://taylor_description/meshes/caster_wheel.STL; visual mesh filename=package://taylor_description/meshes/caster_wheel.STL
- link left_wheel: geometry collision mesh filename=package://taylor_description/meshes/left_wheel.STL; visual mesh filename=package://taylor_description/meshes/left_wheel.STL
- link lidar: geometry collision mesh filename=package://taylor_description/meshes/lidar.STL; visual mesh filename=package://taylor_description/meshes/lidar.STL
- link right_wheel: geometry collision mesh filename=package://taylor_description/meshes/right_wheel.STL; visual mesh filename=package://taylor_description/meshes/right_wheel.STL
