Commit message: [fix] URDF working

File: taylor_robot_description/urdf/gazebo_control.xacro (robot description, xacro)
@@ -6,6 +6,6 @@
             <left_joint>left_wheel_joint</left_joint>
             <right_joint>right_wheel_joint</right_joint>
-            <wheel_separation>0.40</wheel_separation>
-            <wheel_diameter>0.1</wheel_diameter>
+            <wheel_separation>0.15</wheel_separation>
+            <wheel_diameter>0.06</wheel_diameter>
             <!-- Limits -->
             <max_wheel_torque>200</max_wheel_torque>

File: taylor_robot_description/urdf/taylor.robot.core.xacro (robot description, xacro)
@@ -4,11 +4,5 @@
      For more information, please see http://wiki.ros.org/sw_urdf_exporter -->
 <robot xmlns:xacro="http://www.ros.org/wiki/xacro" name="taylor_robot_description">
-  <link name="base_link"/>
-  <joint name="chassis_joint" type="fixed">
-    <parent link="base_link"/>
-    <child link="chassis_link"/>
-    <origin xyz="0 0.0 0.0"/>
-  </joint>
-  <link name="chassis_link">
+    <link name="chassis_link">
     <inertial>
       <origin xyz="0.097174 0.025101 1.9337E-06" rpy="0 0 0"/>
@@ -26,7 +20,5 @@
       <origin xyz="0 0 0" rpy="0 0 0" />
       <geometry>
-        <mesh>
-          <uri>model://taylor_robot_description/meshes/chassis_link.STL</uri>
-        </mesh>
+        <mesh filename="file://$(find taylor_robot_description)/meshes/chassis_link.STL" scale="1 1 1" />
       </geometry>
       <material name="">
@@ -37,7 +29,5 @@
       <origin xyz="0 0 0" rpy="0 0 0" />
       <geometry>
-        <mesh>
-         <uri>model://taylor_robot_description/meshes/chassis_link.STL</uri>
-        </mesh>
+        <mesh filename="file://$(find taylor_robot_description)/meshes/chassis_link.STL" scale="1 1 1" />
       </geometry>
     </collision>
@@ -63,7 +53,5 @@
         rpy="0 0 0" />
       <geometry>
-        <mesh>
-          <uri>model://taylor_robot_description/meshes/right_wheel.STL</uri>
-        </mesh>
+        <mesh filename="file://$(find taylor_robot_description)/meshes/right_wheel.STL" scale="1 1 1" />
       </geometry>
       <material
@@ -78,7 +66,5 @@
         rpy="0 0 0" />
       <geometry>
-        <mesh>
-          <uri>model://taylor_robot_description/meshes/right_wheel.STL</uri>
-        </mesh>
+        <mesh filename="file://$(find taylor_robot_description)/meshes/right_wheel.STL" scale="1 1 1" />
       </geometry>
     </collision>
@@ -90,5 +76,5 @@
       rpy="1.5708 0 1.5708" />
     <parent
-      link="base_link" />
+      link="chassis_link" />
     <child
       link="right_wheel" />
@@ -116,7 +102,5 @@
         rpy="0 0 0" />
       <geometry>
-        <mesh>
-         <uri>model://taylor_robot_description/meshes/left_wheel.STL</uri>
-        </mesh>
+        <mesh filename="file://$(find taylor_robot_description)/meshes/left_wheel.STL" scale="1 1 1" />
       </geometry>
       <material
@@ -131,7 +115,5 @@
         rpy="0 0 0" />
       <geometry>
-        <mesh>
-          <uri>model://taylor_robot_description/meshes/left_wheel.STL</uri>
-        </mesh>
+        <mesh filename="file://$(find taylor_robot_description)/meshes/left_wheel.STL" scale="1 1 1" />
       </geometry>
     </collision>
@@ -143,5 +125,5 @@
       rpy="1.5708 0 1.5708" />
     <parent
-      link="base_link" />
+      link="chassis_link" />
     <child
       link="left_wheel" />
@@ -169,7 +151,5 @@
         rpy="0 0 0" />
       <geometry>
-        <mesh>
-          <uri>model://taylor_robot_description/meshes/caster_wheel.STL</uri>
-        </mesh>
+        <mesh filename="file://$(find taylor_robot_description)/meshes/caster_wheel.STL" scale="1 1 1" />
       </geometry>
       <material
@@ -184,12 +164,10 @@
         rpy="0 0 0" />
       <geometry>
-        <mesh>
-          <uri>model://taylor_robot_description/meshes/caster_wheel.STL</uri>
-        </mesh>
+        <mesh filename="file://$(find taylor_robot_description)/meshes/caster_wheel.STL" scale="1 1 1" />
       </geometry>
     </collision>
   </link>
   <joint name="caster_wheel_joint"
-    type="continuous">
+    type="fixed">
     <origin
       xyz="0.17 0 -0.009"
@@ -222,7 +200,5 @@
         rpy="0 0 0" />
       <geometry>
-        <mesh>
-          <uri>package://taylor_robot_description/meshes/lidar.STL</uri>
-        </mesh>
+        <mesh filename="file://$(find taylor_robot_description)/meshes/lidar.STL" scale="1 1 1" />
       </geometry>
       <material
@@ -237,7 +213,5 @@
         rpy="0 0 0" />
       <geometry>
-        <mesh>
-          <uri>package://taylor_robot_description/meshes/lidar.STL</uri>
-        </mesh>
+        <mesh filename="file://$(find taylor_robot_description)/meshes/lidar.STL" scale="1 1 1" />
       </geometry>
     </collision>
@@ -255,3 +229,19 @@
       xyz="0 0 0" />
   </joint>
+  <gazebo reference="caster_wheel">
+    <mu1 value="0.001"/>
+    <mu2 value="0.001"/>
+  </gazebo>
+  <gazebo reference="right_wheel">
+    <material>Gazebo/Black</material>
+  </gazebo>
+  <gazebo reference="left_wheel">
+    <material>Gazebo/Black</material>
+  </gazebo>
+  <gazebo reference="lidar">
+    <material>Gazebo/Black</material>
+  </gazebo>
+  <gazebo reference="chassis_link">
+    <material>Gazebo/Purple</material>
+  </gazebo>
 </robot>
