Commit message: [change] Trying to make the URDF work

File: taylor_robot_description/urdf/taylor.robot.core.xacro (robot description, xacro)
@@ -3,14 +3,15 @@
      Commit Version: 1.6.0-4-g7f85cfe  Build Version: 1.6.7995.38578
      For more information, please see http://wiki.ros.org/sw_urdf_exporter -->
-<robot
-  name="taylor_description">
-  <link
-    name="base_link">
-    <inertial>
-      <origin
-        xyz="0.097174 0.025101 1.9337E-06"
-        rpy="0 0 0" />
-      <mass
-        value="0.65385" />
+<robot xmlns:xacro="http://www.ros.org/wiki/xacro" name="taylor_robot_description">
+  <link name="base_link"/>
+  <joint name="chassis_joint" type="fixed">
+    <parent link="base_link"/>
+    <child link="chassis_link"/>
+    <origin xyz="0 0.0 0.0"/>
+  </joint>
+  <link name="chassis_link">
+    <inertial>
+      <origin xyz="0.097174 0.025101 1.9337E-06" rpy="0 0 0"/>
+      <mass value="0.65385" />
       <inertia
         ixx="0.002038"
@@ -19,32 +20,28 @@
         iyy="0.0059638"
         iyz="-1.9482E-08"
-        izz="0.0043786" />
-    </inertial>
-    <visual>
-      <origin
-        xyz="0 0 0"
-        rpy="0 0 0" />
-      <geometry>
-        <mesh
-          filename="package://taylor_description/meshes/base_link.STL" />
-      </geometry>
-      <material
-        name="">
-        <color
-          rgba="0.79216 0.81961 0.93333 1" />
-      </material>
-    </visual>
-    <collision>
-      <origin
-        xyz="0 0 0"
-        rpy="0 0 0" />
-      <geometry>
-        <mesh
-          filename="package://taylor_description/meshes/base_link.STL" />
-      </geometry>
-    </collision>
-  </link>
-  <link
-    name="right_wheel">
+        izz="0.0043786"
+      />
+    </inertial>
+    <visual>
+      <origin xyz="0 0 0" rpy="0 0 0" />
+      <geometry>
+        <mesh>
+          <uri>model://taylor_robot_description/meshes/chassis_link.STL</uri>
+        </mesh>
+      </geometry>
+      <material name="">
+        <color rgba="0.79216 0.81961 0.93333 1" />
+      </material>
+    </visual>
+    <collision>
+      <origin xyz="0 0 0" rpy="0 0 0" />
+      <geometry>
+        <mesh>
+         <uri>model://taylor_robot_description/meshes/chassis_link.STL</uri>
+        </mesh>
+      </geometry>
+    </collision>
+  </link>
+  <link name="right_wheel">
     <inertial>
       <origin
@@ -66,6 +63,7 @@
         rpy="0 0 0" />
       <geometry>
-        <mesh
-          filename="package://taylor_description/meshes/right_wheel.STL" />
+        <mesh>
+          <uri>model://taylor_robot_description/meshes/right_wheel.STL</uri>
+        </mesh>
       </geometry>
       <material
@@ -80,11 +78,11 @@
         rpy="0 0 0" />
       <geometry>
-        <mesh
-          filename="package://taylor_description/meshes/right_wheel.STL" />
-      </geometry>
-    </collision>
-  </link>
-  <joint
-    name="right_wheel_joint"
+        <mesh>
+          <uri>model://taylor_robot_description/meshes/right_wheel.STL</uri>
+        </mesh>
+      </geometry>
+    </collision>
+  </link>
+  <joint name="right_wheel_joint"
     type="continuous">
     <origin
@@ -98,6 +96,5 @@
       xyz="1 0 0" />
   </joint>
-  <link
-    name="left_wheel">
+  <link name="left_wheel">
     <inertial>
       <origin
@@ -119,6 +116,7 @@
         rpy="0 0 0" />
       <geometry>
-        <mesh
-          filename="package://taylor_description/meshes/left_wheel.STL" />
+        <mesh>
+         <uri>model://taylor_robot_description/meshes/left_wheel.STL</uri>
+        </mesh>
       </geometry>
       <material
@@ -133,11 +131,11 @@
         rpy="0 0 0" />
       <geometry>
-        <mesh
-          filename="package://taylor_description/meshes/left_wheel.STL" />
-      </geometry>
-    </collision>
-  </link>
-  <joint
-    name="left_wheel_joint"
+        <mesh>
+          <uri>model://taylor_robot_description/meshes/left_wheel.STL</uri>
+        </mesh>
+      </geometry>
+    </collision>
+  </link>
+  <joint name="left_wheel_joint"
     type="continuous">
     <origin
@@ -151,6 +149,5 @@
       xyz="1 0 0" />
   </joint>
-  <link
-    name="caster_wheel">
+  <link name="caster_wheel">
     <inertial>
       <origin
@@ -172,6 +169,7 @@
         rpy="0 0 0" />
       <geometry>
-        <mesh
-          filename="package://taylor_description/meshes/caster_wheel.STL" />
+        <mesh>
+          <uri>model://taylor_robot_description/meshes/caster_wheel.STL</uri>
+        </mesh>
       </geometry>
       <material
@@ -186,11 +184,11 @@
         rpy="0 0 0" />
       <geometry>
-        <mesh
-          filename="package://taylor_description/meshes/caster_wheel.STL" />
-      </geometry>
-    </collision>
-  </link>
-  <joint
-    name="caster_wheel_joint"
+        <mesh>
+          <uri>model://taylor_robot_description/meshes/caster_wheel.STL</uri>
+        </mesh>
+      </geometry>
+    </collision>
+  </link>
+  <joint name="caster_wheel_joint"
     type="continuous">
     <origin
@@ -198,5 +196,5 @@
       rpy="1.5708 0 -0.16473" />
     <parent
-      link="base_link" />
+      link="chassis_link" />
     <child
       link="caster_wheel" />
@@ -204,6 +202,5 @@
       xyz="0 1 0" />
   </joint>
-  <link
-    name="lidar">
+  <link name="lidar">
     <inertial>
       <origin
@@ -225,6 +222,7 @@
         rpy="0 0 0" />
       <geometry>
-        <mesh
-          filename="package://taylor_description/meshes/lidar.STL" />
+        <mesh>
+          <uri>package://taylor_robot_description/meshes/lidar.STL</uri>
+        </mesh>
       </geometry>
       <material
@@ -239,11 +237,11 @@
         rpy="0 0 0" />
       <geometry>
-        <mesh
-          filename="package://taylor_description/meshes/lidar.STL" />
-      </geometry>
-    </collision>
-  </link>
-  <joint
-    name="lidar_joint"
+        <mesh>
+          <uri>package://taylor_robot_description/meshes/lidar.STL</uri>
+        </mesh>
+      </geometry>
+    </collision>
+  </link>
+  <joint name="lidar_joint"
     type="fixed">
     <origin
@@ -251,5 +249,5 @@
       rpy="1.5708 0 0" />
     <parent
-      link="base_link" />
+      link="chassis_link" />
     <child
       link="lidar" />

Commit message: [add] Basic ros2_control files

File: taylor_robot_description/urdf/taylor.robot.core.xacro (robot description, xacro)
@@ -229,19 +229,3 @@
       xyz="0 0 0" />
   </joint>
-  <gazebo reference="caster_wheel">
-    <mu1 value="0.001"/>
-    <mu2 value="0.001"/>
-  </gazebo>
-  <gazebo reference="right_wheel">
-    <material>Gazebo/Black</material>
-  </gazebo>
-  <gazebo reference="left_wheel">
-    <material>Gazebo/Black</material>
-  </gazebo>
-  <gazebo reference="lidar">
-    <material>Gazebo/Black</material>
-  </gazebo>
-  <gazebo reference="chassis_link">
-    <material>Gazebo/Purple</material>
-  </gazebo>
 </robot>

Commit message: [change] Trying to fix some bugs

File: taylor_robot_description/urdf/taylor.robot.core.xacro (robot description, xacro)
@@ -4,4 +4,5 @@
      For more information, please see http://wiki.ros.org/sw_urdf_exporter -->
 <robot xmlns:xacro="http://www.ros.org/wiki/xacro" name="taylor_robot_description">
+  <xacro:macro name="taylor" params="prefix">
     <link name="chassis_link">
     <inertial>
@@ -229,3 +230,20 @@
       xyz="0 0 0" />
   </joint>
+  <gazebo reference="caster_wheel">
+    <mu1 value="0.001"/>
+    <mu2 value="0.001"/>
+  </gazebo>
+  <gazebo reference="right_wheel">
+    <material>Gazebo/Black</material>
+  </gazebo>
+  <gazebo reference="left_wheel">
+    <material>Gazebo/Black</material>
+  </gazebo>
+  <gazebo reference="lidar">
+    <material>Gazebo/Black</material>
+  </gazebo>
+  <gazebo reference="chassis_link">
+    <material>Gazebo/Purple</material>
+  </gazebo>
+</xacro:macro>
 </robot>

File: taylor_robot_description/urdf/taylor.robot.urdf.xacro (robot description, xacro)
@@ -2,7 +2,7 @@
 <robot xmlns:xacro="http://www.ros.org/wiki/xacro" name="taylor_robot">
   <xacro:arg name="prefix" default=""/>
-  <xacro:include filename="$(find taylor_robot_description)/urdf/taylor.robot.core.xacro"/>
-  <xacro:include filename="$(find taylor_robot_description)/gazebo/taylor.gazebo.xacro"/>
+  <xacro:include filename="$(find taylor_robot_description)/gazebo/taylor.materials.xacro"/>
   <xacro:include filename="$(find taylor_robot_description)/urdf/taylor.lidar.xacro"/>
+  <xacro:taylor prefix="$(arg prefix)"/>
   <xacro:taylor_ros2_control name="Taylor" prefix="$(arg prefix)"/>
 </robot>

Commit message: [removed] wrong models were excluded from lab_25 file

File: taylor_robot_description/urdf/taylor.robot.core.xacro (robot description, xacro)
@@ -244,5 +244,5 @@
   </gazebo>
   <gazebo reference="chassis_link">
-    <material>Gazebo/Purple</material>
+    <material>Gazebo/Red</material>
   </gazebo>
 </xacro:macro>
