Commit message: [change] Chassis_link to base_link for nav2 works

File: taylor_robot/gazebo/gazebo_control.xacro (robot description, xacro)
@@ -13,5 +13,5 @@
             <!-- Output -->
             <odometry_frame>odom</odometry_frame>
-            <robot_base_frame>chassis_link</robot_base_frame>
+            <robot_base_frame>base_link</robot_base_frame>
             <publish_odom>true</publish_odom>
             <publish_odom_tf>true</publish_odom_tf>

File: taylor_robot/gazebo/taylor.gazebo.xacro (robot description, xacro)
@@ -14,5 +14,5 @@
         <material>Gazebo/Black</material>
     </gazebo>
-    <gazebo reference="chassis_link">
+    <gazebo reference="base_link">
         <material>Gazebo/White</material>
     </gazebo>

File: taylor_robot/urdf/taylor.robot.core.xacro (robot description, xacro)
@@ -6,5 +6,5 @@
   <xacro:macro name="taylor" params="prefix">
     <link name="base_footprint"/>
-    <link name="chassis_link">
+    <link name="base_link">
     <inertial>
       <origin xyz="0.097174 0.025101 1.9337E-06" rpy="0 0 0"/>
@@ -22,5 +22,5 @@
       <origin xyz="0 0 0" rpy="0 0 0" />
       <geometry>
-        <mesh filename="file://$(find taylor_robot)/meshes/chassis_link.STL" scale="1 1 1" />
+        <mesh filename="file://$(find taylor_robot)/meshes/base_link.STL" scale="1 1 1" />
       </geometry>
       <material name="">
@@ -31,10 +31,10 @@
       <origin xyz="0 0 0" rpy="0 0 0" />
       <geometry>
-        <mesh filename="file://$(find taylor_robot)/meshes/chassis_link.STL" scale="1 1 1" />
+        <mesh filename="file://$(find taylor_robot)/meshes/base_link.STL" scale="1 1 1" />
       </geometry>
     </collision>
   </link>
   <joint name="base_joint" type="fixed">
-      <parent link="chassis_link"/>
+      <parent link="base_link"/>
       <child link="base_footprint"/>
       <origin xyz="0 0 0" rpy="0 0 0"/>
@@ -83,5 +83,5 @@
       rpy="1.5708 0 1.5708" />
     <parent
-      link="chassis_link" />
+      link="base_link" />
     <child
       link="right_wheel" />
@@ -132,5 +132,5 @@
       rpy="1.5708 0 1.5708" />
     <parent
-      link="chassis_link" />
+      link="base_link" />
     <child
       link="left_wheel" />
@@ -181,5 +181,5 @@
       rpy="1.5708 0 -0.16473" />
     <parent
-      link="chassis_link" />
+      link="base_link" />
     <child
       link="caster_wheel" />
@@ -230,5 +230,5 @@
       rpy="1.5708 0 0" />
     <parent
-      link="chassis_link" />
+      link="base_link" />
     <child
       link="lidar" />
