Commit message: [change] Change taylor's colors

File: taylor_robot/gazebo/taylor.gazebo.xacro (robot description, xacro)
@@ -15,5 +15,10 @@
     </gazebo>
     <gazebo reference="chassis_link">
-        <material>Gazebo/Purple</material>
+        <material>Gazebo/White</material>
+    </gazebo>
+    <gazebo reference="caster_wheel">
+        <material>Gazebo/Black</material>
+        <mu0 value="0.001"/>
+        <mu1 value="0.001"/>
     </gazebo>
 </robot>

File: taylor_robot/urdf/taylor.robot.core.xacro (robot description, xacro)
@@ -230,20 +230,4 @@
       xyz="0 0 0" />
   </joint>
-  <gazebo reference="caster_wheel">
-    <mu1 value="0.001"/>
-    <mu2 value="0.001"/>
-  </gazebo>
-  <gazebo reference="right_wheel">
-    <material>Gazebo/Black</material>
-  </gazebo>
-  <gazebo reference="left_wheel">
-    <material>Gazebo/Black</material>
-  </gazebo>
-  <gazebo reference="lidar">
-    <material>Gazebo/Black</material>
-  </gazebo>
-  <gazebo reference="chassis_link">
-    <material>Gazebo/Red</material>
-  </gazebo>
-</xacro:macro>
+  </xacro:macro>
 </robot>

File: taylor_robot/urdf/taylor.robot.urdf.xacro (robot description, xacro)
@@ -3,5 +3,5 @@
   <xacro:arg name="prefix" default=""/>
   <xacro:include filename="$(find taylor_robot)/gazebo/gazebo_control.xacro"/>
-  <xacro:include filename="$(find taylor_robot)/gazebo/taylor.materials.xacro"/>
+  <xacro:include filename="$(find taylor_robot)/gazebo/taylor.gazebo.xacro"/>
   <xacro:include filename="$(find taylor_robot)/urdf/taylor.lidar.xacro"/>
   <xacro:include filename="$(find taylor_robot)/urdf/taylor.robot.core.xacro"/>

Commit message: [added] gazebo plugin and ros2 costmap launch file

File: taylor_robot/gazebo/taylor.gazebo.xacro (robot description, xacro)
@@ -15,5 +15,5 @@
     </gazebo>
     <gazebo reference="chassis_link">
-        <material>Gazebo/Purple</material>
+        <material>Gazebo/Red</material>
     </gazebo>
 </robot>

Commit message: [correction] errors from urdf files are now correct

File: taylor_robot/gazebo/taylor.gazebo.xacro (robot description, xacro)
@@ -2,6 +2,7 @@
 <robot xmlns:xacro="http://ros.org/wiki/xacro">
     <gazebo reference="caster_wheel">
-        <mu1 value="0.001"/>
-        <mu2 value="0.001"/>
+        <mu1 value="0.000001"/>
+        <mu2 value="0.000001"/>
+        <material>Gazebo/Black</material>
     </gazebo>
     <gazebo reference="right_wheel">

File: taylor_robot/urdf/taylor.robot.core.xacro (robot description, xacro)
@@ -5,6 +5,18 @@
 <robot xmlns:xacro="http://www.ros.org/wiki/xacro" name="taylor_robot">
   <xacro:macro name="taylor" params="prefix">
+    <link name="base_link"/>
     <link name="base_footprint"/>
-    <link name="base_link">
+    <joint name="base_joint" type="fixed">
+        <parent link="base_link"/>
+        <child link="base_footprint"/>
+        <origin xyz="0 0 0" rpy="0 0 0"/>
+    </joint>
+    <!-- CHASSIS LINK -->
+    <joint name="chassis_joint" type="fixed">
+        <parent link="base_link"/>
+        <child link="chassis_link"/>
+        <origin xyz="0.0 0.0 0.0"/>
+    </joint>
+    <link name="chassis_link">
     <inertial>
       <origin xyz="0.097174 0.025101 1.9337E-06" rpy="0 0 0"/>
@@ -22,22 +34,15 @@
       <origin xyz="0 0 0" rpy="0 0 0" />
       <geometry>
+        <mesh filename="file://$(find taylor_robot)/meshes/chassis_link.STL" scale="1 1 1" />
+      </geometry>
+      <material name="red"/>
+    </visual>
+    <collision>
+      <origin xyz="0 0 0" rpy="0 0 0" />
+      <geometry>
         <mesh filename="file://$(find taylor_robot)/meshes/base_link.STL" scale="1 1 1" />
       </geometry>
-      <material name="">
-        <color rgba="0.79216 0.81961 0.93333 1" />
-      </material>
-    </visual>
-    <collision>
-      <origin xyz="0 0 0" rpy="0 0 0" />
-      <geometry>
-        <mesh filename="file://$(find taylor_robot)/meshes/base_link.STL" scale="1 1 1" />
-      </geometry>
-    </collision>
-  </link>
-  <joint name="base_joint" type="fixed">
-      <parent link="base_link"/>
-      <child link="base_footprint"/>
-      <origin xyz="0 0 0" rpy="0 0 0"/>
-  </joint>
+    </collision>
+  </link>
   <link name="right_wheel">
     <inertial>
@@ -62,9 +67,5 @@
         <mesh filename="file://$(find taylor_robot)/meshes/right_wheel.STL" scale="1 1 1" />
       </geometry>
-      <material
-        name="">
-        <color
-          rgba="0.792156862745098 0.819607843137255 0.933333333333333 1" />
-      </material>
+      <material name="black"/>
     </visual>
     <collision>
@@ -111,9 +112,5 @@
         <mesh filename="file://$(find taylor_robot)/meshes/left_wheel.STL" scale="1 1 1" />
       </geometry>
-      <material
-        name="">
-        <color
-          rgba="0.792156862745098 0.819607843137255 0.933333333333333 1" />
-      </material>
+      <material name="black"/>
     </visual>
     <collision>
@@ -160,9 +157,5 @@
         <mesh filename="file://$(find taylor_robot)/meshes/caster_wheel.STL" scale="1 1 1" />
       </geometry>
-      <material
-        name="">
-        <color
-          rgba="0.792156862745098 0.819607843137255 0.933333333333333 1" />
-      </material>
+      <material name="black"/>
     </visual>
     <collision>
@@ -209,9 +202,5 @@
         <mesh filename="file://$(find taylor_robot)/meshes/lidar.STL" scale="1 1 1" />
       </geometry>
-      <material
-        name="">
-        <color
-          rgba="1 1 1 1" />
-      </material>
+      <material name="black"/>
     </visual>
     <collision>

File: taylor_robot/urdf/taylor.robot.urdf copy.xacro (robot description, xacro)
@@ -3,8 +3,8 @@
   <xacro:arg name="prefix" default=""/>
   <xacro:include filename="$(find taylor_robot)/gazebo/taylor.gazebo.xacro"/>
-  <xacro:include filename="$(find taylor_robot)/gazebo/taylor.materials.xacro"/>
+  <xacro:include filename="$(find taylor_robot)/urdf/taylor.lidar.xacro"/>
   <xacro:include filename="$(find taylor_robot)/urdf/taylor.robot.core.xacro"/>
-  <xacro:include filename="$(find taylor_robot)/gazebo/gazebo_control.xacro"/>
-  <xacro:include filename="$(find taylor_robot)/urdf/taylor.lidar.xacro"/>
+  <xacro:include filename="$(find taylor_robot)/ros2_control/taylor.ros2_control.xacro"/>
   <xacro:taylor prefix="$(arg prefix)"/>
+  <xacro:taylor_ros2_control name="Taylor" prefix="$(arg prefix)"/>
 </robot>
