Commit message: [fix] rename bugs

File: taylor_robot/urdf/taylor.robot.core.xacro (robot description, xacro)
@@ -3,5 +3,5 @@
      Commit Version: 1.6.0-4-g7f85cfe  Build Version: 1.6.7995.38578
      For more information, please see http://wiki.ros.org/sw_urdf_exporter -->
-<robot xmlns:xacro="http://www.ros.org/wiki/xacro" name="taylor_robot_description">
+<robot xmlns:xacro="http://www.ros.org/wiki/xacro" name="taylor_robot">
   <xacro:macro name="taylor" params="prefix">
     <link name="chassis_link">
@@ -21,5 +21,5 @@
       <origin xyz="0 0 0" rpy="0 0 0" />
       <geometry>
-        <mesh filename="file://$(find taylor_robot_description)/meshes/chassis_link.STL" scale="1 1 1" />
+        <mesh filename="file://$(find taylor_robot)/meshes/chassis_link.STL" scale="1 1 1" />
       </geometry>
       <material name="">
@@ -30,5 +30,5 @@
       <origin xyz="0 0 0" rpy="0 0 0" />
       <geometry>
-        <mesh filename="file://$(find taylor_robot_description)/meshes/chassis_link.STL" scale="1 1 1" />
+        <mesh filename="file://$(find taylor_robot)/meshes/chassis_link.STL" scale="1 1 1" />
       </geometry>
     </collision>
@@ -54,5 +54,5 @@
         rpy="0 0 0" />
       <geometry>
-        <mesh filename="file://$(find taylor_robot_description)/meshes/right_wheel.STL" scale="1 1 1" />
+        <mesh filename="file://$(find taylor_robot)/meshes/right_wheel.STL" scale="1 1 1" />
       </geometry>
       <material
@@ -67,5 +67,5 @@
         rpy="0 0 0" />
       <geometry>
-        <mesh filename="file://$(find taylor_robot_description)/meshes/right_wheel.STL" scale="1 1 1" />
+        <mesh filename="file://$(find taylor_robot)/meshes/right_wheel.STL" scale="1 1 1" />
       </geometry>
     </collision>
@@ -103,5 +103,5 @@
         rpy="0 0 0" />
       <geometry>
-        <mesh filename="file://$(find taylor_robot_description)/meshes/left_wheel.STL" scale="1 1 1" />
+        <mesh filename="file://$(find taylor_robot)/meshes/left_wheel.STL" scale="1 1 1" />
       </geometry>
       <material
@@ -116,5 +116,5 @@
         rpy="0 0 0" />
       <geometry>
-        <mesh filename="file://$(find taylor_robot_description)/meshes/left_wheel.STL" scale="1 1 1" />
+        <mesh filename="file://$(find taylor_robot)/meshes/left_wheel.STL" scale="1 1 1" />
       </geometry>
     </collision>
@@ -152,5 +152,5 @@
         rpy="0 0 0" />
       <geometry>
-        <mesh filename="file://$(find taylor_robot_description)/meshes/caster_wheel.STL" scale="1 1 1" />
+        <mesh filename="file://$(find taylor_robot)/meshes/caster_wheel.STL" scale="1 1 1" />
       </geometry>
       <material
@@ -165,5 +165,5 @@
         rpy="0 0 0" />
       <geometry>
-        <mesh filename="file://$(find taylor_robot_description)/meshes/caster_wheel.STL" scale="1 1 1" />
+        <mesh filename="file://$(find taylor_robot)/meshes/caster_wheel.STL" scale="1 1 1" />
       </geometry>
     </collision>
@@ -201,5 +201,5 @@
         rpy="0 0 0" />
       <geometry>
-        <mesh filename="file://$(find taylor_robot_description)/meshes/lidar.STL" scale="1 1 1" />
+        <mesh filename="file://$(find taylor_robot)/meshes/lidar.STL" scale="1 1 1" />
       </geometry>
       <material
@@ -214,5 +214,5 @@
         rpy="0 0 0" />
       <geometry>
-        <mesh filename="file://$(find taylor_robot_description)/meshes/lidar.STL" scale="1 1 1" />
+        <mesh filename="file://$(find taylor_robot)/meshes/lidar.STL" scale="1 1 1" />
       </geometry>
     </collision>

File: taylor_robot/urdf/taylor.robot.urdf.xacro (robot description, xacro)
@@ -2,8 +2,8 @@
 <robot xmlns:xacro="http://www.ros.org/wiki/xacro" name="taylor_robot">
   <xacro:arg name="prefix" default=""/>
-  <xacro:include filename="$(find taylor_robot_description)/gazebo/taylor.materials.xacro"/>
-  <xacro:include filename="$(find taylor_robot_description)/urdf/taylor.lidar.xacro"/>
-  <xacro:include filename="$(find taylor_robot_description)/urdf/taylor.robot.core.xacro"/>
-  <xacro:include filename="$(find taylor_robot_description)/ros2_control/taylor.ros2_control.xacro"/>
+  <xacro:include filename="$(find taylor_robot)/gazebo/taylor.materials.xacro"/>
+  <xacro:include filename="$(find taylor_robot)/urdf/taylor.lidar.xacro"/>
+  <xacro:include filename="$(find taylor_robot)/urdf/taylor.robot.core.xacro"/>
+  <xacro:include filename="$(find taylor_robot)/ros2_control/taylor.ros2_control.xacro"/>
   <xacro:taylor prefix="$(arg prefix)"/>
   <xacro:taylor_ros2_control name="Taylor" prefix="$(arg prefix)"/>

File: taylor_robot/urdf/taylor_system.urdf.xacro (robot description, xacro)
@@ -11,12 +11,12 @@
   <xacro:arg name="fake_sensor_commands" default="false" />
   <xacro:arg name="prefix" default="" />
-  <xacro:include filename="$(find taylor_robot_description)/urdf/taylor.robot.urdf.xacro" />
-  <xacro:include filename="$(find taylor_robot_description)/gazebo/taylor.materials.xacro" />
+  <xacro:include filename="$(find taylor_robot)/urdf/taylor.robot.urdf.xacro" />
+  <xacro:include filename="$(find taylor_robot)/gazebo/taylor.materials.xacro" />
   <!-- Import all Gazebo-customization elements, including Gazebo colors -->
-  <xacro:include filename="$(find taylor_robot_description)/gazebo/taylor.gazebo.xacro" />
+  <xacro:include filename="$(find taylor_robot)/gazebo/taylor.gazebo.xacro" />
   <!-- Import Rviz colors -->
-  <xacro:include filename="$(find taylor_robot_description)/gazebo/taylor.materials.xacro" />
+  <xacro:include filename="$(find taylor_robot)/gazebo/taylor.materials.xacro" />
   <!-- Import diffbot ros2_control description -->
-  <xacro:include filename="$(find taylor_robot_description)/ros2_control/taylor_system.ros2_control.xacro" />
+  <xacro:include filename="$(find taylor_robot)/ros2_control/taylor_system.ros2_control.xacro" />
   <xacro:taylor_system
     name="TaylorSystem" prefix="$(arg prefix)"

Commit message: [add] base_footprint

File: taylor_robot/urdf/taylor.robot.core.xacro (robot description, xacro)
@@ -5,4 +5,5 @@
 <robot xmlns:xacro="http://www.ros.org/wiki/xacro" name="taylor_robot">
   <xacro:macro name="taylor" params="prefix">
+    <link name="base_footprint"/>
     <link name="chassis_link">
     <inertial>
@@ -34,4 +35,9 @@
     </collision>
   </link>
+  <joint name="base_joint" type="fixed">
+      <parent link="chassis_link"/>
+      <child link="base_footprint"/>
+      <origin xyz="0 0 0" rpy="0 0 0"/>
+  </joint>
   <link name="right_wheel">
     <inertial>

Commit message: [fix] Gazebo not found the models

File: taylor_robot/urdf/taylor.robot.core.xacro (robot description, xacro)
@@ -41,5 +41,5 @@
       <origin xyz="0 0 0" rpy="0 0 0" />
       <geometry>
-        <mesh filename="file://$(find taylor_robot)/meshes/base_link.STL" scale="1 1 1" />
+        <mesh filename="file://$(find taylor_robot)/meshes/chassis_link.STL" scale="1 1 1" />
       </geometry>
     </collision>
