Commit message: organize files and directories

File: description/taylor.robot.core.xacro (robot description, xacro)
@@ -34,5 +34,5 @@
       <origin xyz="0 0 0" rpy="0 0 0" />
       <geometry>
-        <mesh filename="file://$(find taylor_robot)/meshes/chassis_link.STL" scale="1 1 1" />
+        <mesh filename="file://$(find taylor_robot)/description/meshes/chassis_link.STL" scale="1 1 1" />
       </geometry>
       <material name="red"/>
@@ -41,5 +41,5 @@
       <origin xyz="0 0 0" rpy="0 0 0" />
       <geometry>
-        <mesh filename="file://$(find taylor_robot)/meshes/chassis_link.STL" scale="1 1 1" />
+        <mesh filename="file://$(find taylor_robot)/description/meshes/chassis_link.STL" scale="1 1 1" />
       </geometry>
     </collision>
@@ -65,14 +65,14 @@
         rpy="0 0 0" />
       <geometry>
-        <mesh filename="file://$(find taylor_robot)/meshes/right_wheel.STL" scale="1 1 1" />
-      </geometry>
-      <material name="black"/>
-    </visual>
-    <collision>
-      <origin
-        xyz="0 0 0"
-        rpy="0 0 0" />
-      <geometry>
-        <mesh filename="file://$(find taylor_robot)/meshes/right_wheel.STL" scale="1 1 1" />
+        <mesh filename="file://$(find taylor_robot)/description/meshes/right_wheel.STL" scale="1 1 1" />
+      </geometry>
+      <material name="black"/>
+    </visual>
+    <collision>
+      <origin
+        xyz="0 0 0"
+        rpy="0 0 0" />
+      <geometry>
+        <mesh filename="file://$(find taylor_robot)/description/meshes/right_wheel.STL" scale="1 1 1" />
       </geometry>
     </collision>
@@ -110,14 +110,14 @@
         rpy="0 0 0" />
       <geometry>
-        <mesh filename="file://$(find taylor_robot)/meshes/left_wheel.STL" scale="1 1 1" />
-      </geometry>
-      <material name="black"/>
-    </visual>
-    <collision>
-      <origin
-        xyz="0 0 0"
-        rpy="0 0 0" />
-      <geometry>
-        <mesh filename="file://$(find taylor_robot)/meshes/left_wheel.STL" scale="1 1 1" />
+        <mesh filename="file://$(find taylor_robot)/description/meshes/left_wheel.STL" scale="1 1 1" />
+      </geometry>
+      <material name="black"/>
+    </visual>
+    <collision>
+      <origin
+        xyz="0 0 0"
+        rpy="0 0 0" />
+      <geometry>
+        <mesh filename="file://$(find taylor_robot)/description/meshes/left_wheel.STL" scale="1 1 1" />
       </geometry>
     </collision>
@@ -155,14 +155,14 @@
         rpy="0 0 0" />
       <geometry>
-        <mesh filename="file://$(find taylor_robot)/meshes/caster_wheel.STL" scale="1 1 1" />
-      </geometry>
-      <material name="black"/>
-    </visual>
-    <collision>
-      <origin
-        xyz="0 0 0"
-        rpy="0 0 0" />
-      <geometry>
-        <mesh filename="file://$(find taylor_robot)/meshes/caster_wheel.STL" scale="1 1 1" />
+        <mesh filename="file://$(find taylor_robot)/description/meshes/caster_wheel.STL" scale="1 1 1" />
+      </geometry>
+      <material name="black"/>
+    </visual>
+    <collision>
+      <origin
+        xyz="0 0 0"
+        rpy="0 0 0" />
+      <geometry>
+        <mesh filename="file://$(find taylor_robot)/description/meshes/caster_wheel.STL" scale="1 1 1" />
       </geometry>
     </collision>
@@ -200,14 +200,14 @@
         rpy="0 0 0" />
       <geometry>
-        <mesh filename="file://$(find taylor_robot)/meshes/lidar.STL" scale="1 1 1" />
-      </geometry>
-      <material name="black"/>
-    </visual>
-    <collision>
-      <origin
-        xyz="0 0 0"
-        rpy="0 0 0" />
-      <geometry>
-        <mesh filename="file://$(find taylor_robot)/meshes/lidar.STL" scale="1 1 1" />
+        <mesh filename="file://$(find taylor_robot)/description/meshes/lidar.STL" scale="1 1 1" />
+      </geometry>
+      <material name="black"/>
+    </visual>
+    <collision>
+      <origin
+        xyz="0 0 0"
+        rpy="0 0 0" />
+      <geometry>
+        <mesh filename="file://$(find taylor_robot)/description/meshes/lidar.STL" scale="1 1 1" />
       </geometry>
     </collision>

File: description/taylor_system.urdf.xacro (robot description, xacro)
@@ -3,5 +3,5 @@
 <!--
 Copied and modified from ROS1 example -
-https://github.com/ros-simulation/gazebo_ros_demos/blob/kinetic-devel/diffbot_description/urdf/diffbot.xacro
+https://github.com/ros-simulation/gazebo_ros_demos/blob/kinetic-devel/diffbot_description/description/diffbot.xacro
 -->
 <robot xmlns:xacro="http://www.ros.org/wiki/xacro" name="diffdrive_robot">
@@ -11,12 +11,12 @@
   <xacro:arg name="fake_sensor_commands" default="false" />
   <xacro:arg name="prefix" default="" />
-  <xacro:include filename="$(find taylor_robot)/urdf/taylor.robot.urdf.xacro" />
-  <xacro:include filename="$(find taylor_robot)/gazebo/taylor.materials.xacro" />
+  <xacro:include filename="$(find taylor_robot)/description/taylor.robot.urdf.xacro" />
+  <xacro:include filename="$(find taylor_robot)/description/gazebo/taylor.materials.xacro" />
   <!-- Import all Gazebo-customization elements, including Gazebo colors -->
-  <xacro:include filename="$(find taylor_robot)/gazebo/taylor.gazebo.xacro" />
+  <xacro:include filename="$(find taylor_robot)/description/gazebo/taylor.gazebo.xacro" />
   <!-- Import Rviz colors -->
-  <xacro:include filename="$(find taylor_robot)/gazebo/taylor.materials.xacro" />
+  <xacro:include filename="$(find taylor_robot)/description/gazebo/taylor.materials.xacro" />
   <!-- Import diffbot ros2_control description -->
-  <xacro:include filename="$(find taylor_robot)/ros2_control/taylor_system.ros2_control.xacro" />
+  <xacro:include filename="$(find taylor_robot)/description/taylor_system.ros2_control.xacro" />
   <xacro:taylor_system
     name="TaylorSystem" prefix="$(arg prefix)"
