Commit message: [change] remove unnecessary code

File: description/ros2_control.xacro (robot description, xacro)
@@ -1,63 +1,32 @@
 <?xml version="1.0"?>
 <robot xmlns:xacro="http://www.ros.org/wiki/xacro">
-    <xacro:unless value="$(arg sim_mode)">
-        <ros2_control name="RealRobot" type="system">
-            <hardware>
-                <!-- precisamo mudar essses parametros -->
-                <plugin>diffdrive_arduino/DiffDriveArduino</plugin>
-                <param name="left_wheel_name">left_wheel_joint</param>
-                <param name="right_wheel_name">right_wheel_joint</param>
-                <param name="loop_rate">30</param>
-                <param name="device">/dev/ttyUSB0</param>
-                <param name="baud_rate">57600</param>
-                <param name="timeout">1000</param>
-                <param name="enc_counts_per_rev">1497</param>
-            </hardware>
-            <joint name="left_wheel_joint">
-                <command_interface name="velocity">
-                    <param name="min">-10</param>
-                    <param name="max">10</param>
-                </command_interface>
-                <state_interface name="velocity"/>
-                <state_interface name="position"/>
-            </joint>
-            <joint name="right_wheel_joint">
-                <command_interface name="velocity">
-                    <param name="min">-10</param>
-                    <param name="max">10</param>
-                </command_interface>
-                <state_interface name="velocity"/>
-                <state_interface name="position"/>
-            </joint>
-        </ros2_control>
-    </xacro:unless>
-    <xacro:if value="$(arg sim_mode)">
-        <ros2_control name="GazeboSystem" type="system">
-            <hardware>
-                <plugin>gazebo_ros2_control/GazeboSystem</plugin>
-            </hardware>
-            <joint name="left_wheel_joint">
-                <command_interface name="velocity">
-                    <param name="min">-10</param>
-                    <param name="max">10</param>
-                </command_interface>
-                <state_interface name="velocity"/>
-                <state_interface name="position"/>
-            </joint>
-            <joint name="right_wheel_joint">
-                <command_interface name="velocity">
-                    <param name="min">-10</param>
-                    <param name="max">10</param>
-                </command_interface>
-                <state_interface name="velocity"/>
-                <state_interface name="position"/>
-            </joint>
-        </ros2_control>
-    </xacro:if>
-    <gazebo>
-        <plugin name="gazebo_ros2_control" filename="libgazebo_ros2_control.so">
-            <parameters>$(find taylor_robot)/config/my_controllers.yaml</parameters>
-            <parameters>$(find taylor_robot)/config/gaz_ros2_ctl_use_sim.yaml</parameters>
-        </plugin>
-    </gazebo>
+    <ros2_control name="RealRobot" type="system">
+        <hardware>
+            <!-- precisamo mudar essses parametros -->
+            <plugin>diffdrive_arduino/DiffDriveArduino</plugin>
+            <param name="left_wheel_name">left_wheel_joint</param>
+            <param name="right_wheel_name">right_wheel_joint</param>
+            <param name="loop_rate">30</param>
+            <param name="device">/dev/ttyUSB0</param>
+            <param name="baud_rate">57600</param>
+            <param name="timeout">1000</param>
+            <param name="enc_counts_per_rev">1497</param>
+        </hardware>
+        <joint name="left_wheel_joint">
+            <command_interface name="velocity">
+                <param name="min">-10</param>
+                <param name="max">10</param>
+            </command_interface>
+            <state_interface name="velocity"/>
+            <state_interface name="position"/>
+        </joint>
+        <joint name="right_wheel_joint">
+            <command_interface name="velocity">
+                <param name="min">-10</param>
+                <param name="max">10</param>
+            </command_interface>
+            <state_interface name="velocity"/>
+            <state_interface name="position"/>
+        </joint>
+    </ros2_control>
 </robot>

Commit message: [fix] trying to fix gazebo bug

File: description/ros2_control.xacro (robot description, xacro)
@@ -1,32 +1,64 @@
 <?xml version="1.0"?>
 <robot xmlns:xacro="http://www.ros.org/wiki/xacro">
-    <ros2_control name="RealRobot" type="system">
-        <hardware>
-            <!-- precisamo mudar essses parametros -->
-            <plugin>diffdrive_arduino/DiffDriveArduino</plugin>
-            <param name="left_wheel_name">left_wheel_joint</param>
-            <param name="right_wheel_name">right_wheel_joint</param>
-            <param name="loop_rate">30</param>
-            <param name="device">/dev/ttyUSB0</param>
-            <param name="baud_rate">57600</param>
-            <param name="timeout">1000</param>
-            <param name="enc_counts_per_rev">1497</param>
-        </hardware>
-        <joint name="left_wheel_joint">
-            <command_interface name="velocity">
-                <param name="min">-10</param>
-                <param name="max">10</param>
-            </command_interface>
-            <state_interface name="velocity"/>
-            <state_interface name="position"/>
-        </joint>
-        <joint name="right_wheel_joint">
-            <command_interface name="velocity">
-                <param name="min">-10</param>
-                <param name="max">10</param>
-            </command_interface>
-            <state_interface name="velocity"/>
-            <state_interface name="position"/>
-        </joint>
-    </ros2_control>
+    <xacro:unless value="$(arg use_sim_time)">
+        <ros2_control name="RealRobot" type="system">
+            <hardware>
+                <!-- precisamo mudar essses parametros -->
+                <plugin>diffdrive_arduino/DiffDriveArduino</plugin>
+                <param name="left_wheel_name">left_wheel_joint</param>
+                <param name="right_wheel_name">right_wheel_joint</param>
+                <param name="loop_rate">30</param>
+                <param name="device">/dev/ttyUSB0</param>
+                <param name="baud_rate">57600</param>
+                <param name="timeout">1000</param>
+                <param name="enc_counts_per_rev">1497</param>
+            </hardware>
+            <joint name="left_wheel_joint">
+                <command_interface name="velocity">
+                    <param name="min">-10</param>
+                    <param name="max">10</param>
+                </command_interface>
+                <state_interface name="velocity"/>
+                <state_interface name="position"/>
+            </joint>
+            <joint name="right_wheel_joint">
+                <command_interface name="velocity">
+                    <param name="min">-10</param>
+                    <param name="max">10</param>
+                </command_interface>
+                <state_interface name="velocity"/>
+                <state_interface name="position"/>
+            </joint>
+        </ros2_control>
+    </xacro:unless>
+    <xacro:if value="$(arg use_sim_time)">
+        <ros2_control name="GazeboSystem" type="system">
+            <hardware>
+                <plugin>gazebo_ros2_control/GazeboSystem</plugin>
+            </hardware>
+            <joint name="left_wheel_joint">
+                <command_interface name="velocity">
+                    <param name="min">-10</param>
+                    <param name="max">10</param>
+                </command_interface>
+                <state_interface name="velocity"/>
+                <state_interface name="position"/>
+            </joint>
+            <joint name="right_wheel_joint">
+                <command_interface name="velocity">
+                    <param name="min">-10</param>
+                    <param name="max">10</param>
+                </command_interface>
+                <state_interface name="velocity"/>
+                <state_interface name="position"/>
+            </joint>
+        </ros2_control>
+    </xacro:if>
+    <gazebo>
+        <plugin filename="libgazebo_ros2_control.so" name="gazebo_ros2_control" >
+            <robot_param>robot_description</robot_param>
+            <robot_param_node>$(arg namespace)/robot_state_publisher</robot_param_node>
+            <parameters>$(find taylor_robot)/config/my_controllers.yaml</parameters>
+        </plugin>
+    </gazebo>
 </robot>

File: description/taylor.robot.core.xacro (robot description, xacro)
@@ -4,5 +4,6 @@
      For more information, please see http://wiki.ros.org/sw_urdf_exporter -->
 <robot xmlns:xacro="http://www.ros.org/wiki/xacro" name="taylor_robot">
-  <xacro:macro name="taylor" params="prefix">
+  <!-- Implement prefix namespace-->
+  <xacro:macro name="taylor" params="namespace">
     <link name="base_link"/>
     <link name="base_footprint"/>

File: description/taylor.robot.urdf.xacro (robot description, xacro)
@@ -1,17 +1,19 @@
 <?xml version="1.0" encoding="utf-8"?>
 <robot xmlns:xacro="http://www.ros.org/wiki/xacro" name="taylor_robot">
-  <xacro:arg name="prefix" default=""/>
+  <xacro:arg name="namespace" default=""/>
   <xacro:arg name="use_ros2_control" default="true"/>
-  <xacro:arg name="sim_mode" default="false"/>
+  <xacro:arg name="use_sim_time" default="false"/>
+  <xacro:include filename="$(find taylor_robot)/description/gazebo/taylor.gazebo.xacro"/>
+  <xacro:include filename="$(find taylor_robot)/description/gazebo/taylor.materials.xacro"/>
   <xacro:include filename="$(find taylor_robot)/description/taylor.robot.core.xacro"/>
+  <!-- Use only ros2_control if it's not a simulation, otherwise uses ros2_control + gazebo_ros2_control plugin-->
   <xacro:if value="$(arg use_ros2_control)">
     <xacro:include filename="$(find taylor_robot)/description/ros2_control.xacro"/>
   </xacro:if>
+  <!-- Use diff plugin from gazebo to control the robot -->
   <xacro:unless value="$(arg use_ros2_control)">
-    <xacro:include filename="$(find taylor_robot)/description/gazebo/taylor.gazebo.xacro"/>
-    <xacro:include filename="$(find taylor_robot)/description/gazebo/taylor.materials.xacro"/>
     <xacro:include filename="$(find taylor_robot)/description/gazebo/gazebo_control.xacro"/>
   </xacro:unless>
   <xacro:include filename="$(find taylor_robot)/description/taylor.lidar.xacro"/>
-  <xacro:taylor prefix="$(arg prefix)"/>
+  <xacro:taylor namespace="$(arg namespace)"/>
 </robot>
