Commit message: [create] ros2 -> nav2 interface was created for real taylor_robot

File: description/taylor.lidar.xacro (robot description, xacro)
@@ -4,5 +4,5 @@
         <parent link="lidar"/>
         <child link="laser_frame"/>
-        <origin xyz="0 0 0" rpy="${pi/2} 0 0"/>
+        <origin xyz="0 0 0" rpy="${-pi/2} 0 0"/>
     </joint>
     <link name="laser_frame"/>

File: description/taylor.robot.core.xacro (robot description, xacro)
@@ -217,5 +217,5 @@
     <origin
       xyz="0.034828 0 0.0936"
-      rpy="-1.5708 0 0" />
+      rpy="${pi/2}  0 0" />
     <parent
       link="base_link" />
